File: pcb_left/simple_split_v1.kicad_pcb (KiCad board)
At the start: 2 copper layers, 151.1 x 148.4 mm, 59 parts

Commit message: Update: pcbs routed
Routing:
- net middle_top: track 21.2 -> 35.7 mm
Changed lines of the file:
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@@
+	)
+	(segment
+		(start 206.15 101.5)
+		(end 208.31 101.5)
+		(width 0.2)
+		(layer "F.Cu")
+		(net 20)
 	)
 	(segment
@@
 		(start 205.475 95.075)
 		(end 204.5 95.075)
-		(width 0.2)
-		(layer "F.Cu")
-		(net 20)
-	)
-	(segment
-		(start 206.15 101.5)
-		(end 208.31 101.5)
 		(width 0.2)
 		(layer "F.Cu")
@@
 	)
 	(segment
+		(start 199.101 97.601)
+		(end 198.076 97.601)
+		(width 0.2)
+		(layer "B.Cu")
+		(net 20)
+	)
+	(segment
+		(start 206.15 101.5)
+		(end 205.249 100.599)
+		(width 0.2)
+		(layer "B.Cu")
+		(net 20)
+	)
+	(segment
+		(start 206.15 101.5)
+		(end 208.31 101.5)
+		(width 0.2)
+		(layer "B.Cu")
+		(net 20)
+	)
+	(segment
 		(start 202.359834 93.896)
 		(end 203.538834 95.075)
@@
 	)
 	(segment
+		(start 202.099 100.599)
+		(end 199.101 97.601)
+		(width 0.2)
+		(layer "B.Cu")
+		(net 20)
+	)
+	(segment
 		(start 198.079 93.896)
 		(end 202.359834 93.896)
 		(width 0.2)
 		(layer "B.Cu")
+		(net 20)
+	)
+	(segment
+		(start 205.249 100.599)
+		(end 202.099 100.599)
+		(width 0.2)
+		(layer "B.Cu")
+		(net 20)
+	)
+	(segment
+		(start 198.076 97.601)
+		(end 196.225 95.75)
+		(width 0.2)
+		(layer "B.Cu")
